Commit message: Create for Hoang a Ticket for Docking, Refreshed Metrics Documentation

File: catkin_ws/src/amr_description/urdf/xstack_amr.urdf (robot description, URDF)
Before this commit: robot xstack_amr, 15 links, 14 joints
Links:
- link mast_link: mass 6.0 -> 6.5; geometry collision box size=0.06 0.32 0.90; visual box size=0.06 0.32 0.90
Joints:
- joint lift_joint: limit lower=-0.02 upper=0.75 effort=1500.0 velocity=0.12 -> lower=-0.02 upper=0.80 effort=1500.0 velocity=0.12
