Commit message: Rack-leg docking, height-based lift and pick inventory for XStack
- pallet_detect: detect_rack_legs() finds the bay from the two floor
  runners under the bottom plank, so full and empty bays look the same
- milestone2_mission: detect_mode (rack_legs default, load_face legacy);
  lift heights from the exported pallet height (entry -40 mm, rise 50 mm);
  pick units (lower pallet takes its stack) recorded in
  /warehouse_inventory/empty, empty slots refused; reset_inventory arg
- URDF mast 1.25 m / lift 1.15 m; new NewMapnoObs map as xstack default;
  re-exported locations_milestone_3.yaml
- tests: rack-leg detection (full/empty bay, rotation, 181 rays) and
  pick units on the exported layout

Co-Authored-By: Claude Opus 5.5 <noreply@anthropic.com>

File: catkin_ws/src/amr_description/urdf/xstack_amr.urdf (robot description, URDF)
Before this commit: robot xstack_amr, 15 links, 14 joints
Links:
- link mast_link: geometry collision box size=0.06 0.32 1.25; visual box size=0.06 0.32 1.25
Joints:
- joint lift_joint: limit lower=-0.02 upper=0.80 effort=1500.0 velocity=0.12 -> lower=-0.02 upper=1.15 effort=1500.0 velocity=0.12
